File: PPDuino_Nano_Electronic/PPDuino Nano Procesador/PPDuino_Nano_Procesador.kicad_pcb (KiCad board)
At the start: 2 copper layers, 39.7 x 71.8 mm, 9 parts, among them J1 PWR_IN, J11 INPUTS, J12 OUTPUTS, J2 Conn_01x12, U1 L7805, U6 +5V

Commit message: PCB Complete
Parts:
- added REF**: MountingHole_3.2mm_M3, MountingHole:MountingHole_3.2mm_M3, F.Cu at (114.4, 75.2)
Routing:
- net VDD: track 105.7 -> 119.6 mm
- net GND: track 144.1 -> 155.9 mm
- net +5V: track 157.5 -> 162.5 mm
- net GND1: track 104.5 -> 107.6 mm
- added copper zone on B.Cu, net (none)
