File: PPDuino_Nano_Electronic/PPDuino Nano Entradas/PPDuino Nano Entradas.kicad_sch (KiCad schematic)
At the start: 26 parts, among them J10 PWR_OUT, J11 INPUTS, J2 DI, J3 AI, U1 4N35, U2 4N35, U3 4N35, U4 4N35

Commit message: Actualizar documentacion 2
Other:
- note added: "CONECTORES"
- note added: "INDICADOR DE ALIMENTACION"
- moved on the sheet: D1, D2, D3, D4, D5, J10, J11, J2, J3, R1, R10, R11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
