File: PPDuino_Nano_Electronic/PPDuino Nano Salidas/PPDuino Nano Salidas.kicad_pcb (KiCad board)
At the start: 2 copper layers, 51.6 x 92.8 mm, 28 parts, among them J12 OUTPUTS, J13 SEL1, J14 RLY0, J6 SEL0, J7 RLY1, J8 PWM, J9 PWR_OUT, Q1 BC548, Q2 BC548, U5 L293D

Commit message: PCB Complete
Parts:
- added REF**: MountingHole_3.2mm_M3, MountingHole:MountingHole_3.2mm_M3, F.Cu at (107.4, 65.3)
- moved J13 3.30 mm to (113.1, 100.9)
- moved U5 2.08 mm to (80.0, 58.8)
- moved D8 0.85 mm to (120.2, 76.2)
- moved J6 0.85 mm to (100.8, 101.2)
- moved K1 0.85 mm to (94.5, 88.4)
- moved Q2 0.85 mm to (108.9, 76.7)
- moved R14 0.85 mm to (93.2, 72.2)
- moved R15 0.85 mm to (112.4, 72.0)
- moved D6 0.85 mm to (100.8, 75.8)
- moved K2 0.85 mm to (113.8, 88.5)
- moved Q1 0.85 mm to (89.6, 76.5)
Connections:
- J12 pad 1: GND1 -> GND
Routing:
- net GND: track 76.0 -> 249.0 mm, vias 2 -> 6
- net VDD: track 0.00 -> 122.0 mm, vias 0 -> 4
- net /PWM2m: track 13.3 -> 107.1 mm
- net /PWM3m: track 25.0 -> 114.1 mm
- net /PWM0m: track 31.9 -> 88.5 mm, vias 0 -> 2
- net Net-(D5-K): track 3.92 -> 59.7 mm
- net +5V: track 120.5 -> 174.5 mm, vias 6 -> 10
- net /PWM1m: track 44.9 -> 98.2 mm, vias 2 -> 4
- net Net-(D7-K): track 9.41 -> 52.7 mm, vias 0 -> 2
- net /PWM3: track 110.6 -> 128.1 mm
- net Net-(J14-Pin_2): track 44.6 -> 57.4 mm
- net Net-(J6-Pin_3): track 0.00 -> 11.7 mm
- net Net-(J6-Pin_1): track 0.00 -> 7.12 mm
- net /PWM2: track 107.9 -> 110.7 mm, vias 2 -> 0
- net Net-(J13-Pin_1): track 8.36 -> 10.3 mm
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- added copper zone on B.Cu, net (none)

Commit message: Actualizar documentacion 2
Parts:
- moved D6 46.5 mm to (147.1, 80.9)
- moved Q1 46.5 mm to (135.8, 81.6)
- moved R15 46.5 mm to (158.6, 77.0)
- moved D10 46.5 mm to (140.5, 123.1)
- moved D5 46.5 mm to (153.4, 123.1)
- moved D7 46.5 mm to (163.5, 123.2)
- moved D8 46.5 mm to (166.4, 81.2)
- moved J12 46.5 mm to (155.0, 45.9)
- moved J14 46.5 mm to (150.9, 131.8)
- moved J7 46.5 mm to (161.0, 131.8)
- moved J8 46.5 mm to (130.6, 131.9)
- moved J9 46.5 mm to (120.5, 131.8)
- moved K1 46.5 mm to (140.8, 93.5)
- moved R13 46.5 mm to (153.4, 118.3)
- moved R14 46.5 mm to (139.4, 77.2)
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