File: PPDuino_Nano_Electronic/V0.2/Entradas/PPDuino Nano Entradas.kicad_pcb (KiCad board)
At the start: 2 copper layers, 51.6 x 59.4 mm, 27 parts, among them J10 PWR_OUT, J11 INPUTS, J2 DI, J3 AI, U1 4N35, U2 4N35, U3 4N35, U4 4N35

Commit message: PCB V0.2
Parts:
- removed U1, U2, U3, U4: 4N35, Package_DIP:DIP-6_W7.62mm_LongPads
- added D6: Z5.1V, Diode_THT:D_DO-35_SOD27_P7.62mm_Horizontal, F.Cu at (169.6, 88.8)
- added D7: Z5.1V, Diode_THT:D_DO-35_SOD27_P7.62mm_Horizontal, F.Cu at (166.8, 88.8)
- added G***: LOGO, Logo PPDuino Nano:Logo PPDuino Nano, F.Cu at (124.4, 85.0)
- added G***: LOGO, Logo Fab Lab PPD Electronica:Logo Fab Lab PPD Electronica, F.Cu at (165.7, 109.0)
- added G***: LOGO, Logo Fab Lab PPD Electronica:Logo Fab Lab PPD Electronica, B.Cu at (132.3, 104.7)
- added G***: LOGO, Logo PPDuino Nano:Logo PPDuino Nano, B.Cu at (156.2, 104.6)
- added Q1: BC548, Package_TO_SOT_THT:TO-92L_Inline_Wide, F.Cu at (133.4, 93.5)
- added Q2: BC548, Package_TO_SOT_THT:TO-92L_Inline_Wide, F.Cu at (141.1, 93.5)
- added Q3: BC548, Package_TO_SOT_THT:TO-92L_Inline_Wide, F.Cu at (148.7, 93.5)
- added Q4: BC548, Package_TO_SOT_THT:TO-92L_Inline_Wide, F.Cu at (156.2, 93.5)
- added R14: 2.2k, Resistor_THT:R_Axial_DIN0207_L6.3mm_D2.5mm_P7.62mm_Horizontal, F.Cu at (160.3, 91.9)
- added R15: 2.2k, Resistor_THT:R_Axial_DIN0207_L6.3mm_D2.5mm_P7.62mm_Horizontal, F.Cu at (160.3, 81.3)
- added R16: 2.2k, Resistor_THT:R_Axial_DIN0207_L6.3mm_D2.5mm_P7.62mm_Horizontal, F.Cu at (163.6, 91.9)
- added R17: 2.2k, Resistor_THT:R_Axial_DIN0207_L6.3mm_D2.5mm_P7.62mm_Horizontal, F.Cu at (163.6, 81.3)
- D1: value DI3 -> DI0
- D2: value DI2 -> DI1
- D3: value DI1 -> DI2
- D4: value DI0 -> DI3
- moved D4 15.0 mm to (148.4, 74.8)
- moved D1 15.0 mm to (133.4, 74.7)
- moved R3 11.4 mm to (151.1, 106.5), turned to 90 degrees
- moved R6 8.77 mm to (143.6, 106.5), turned to 90 degrees
- moved R11 6.31 mm to (135.9, 106.5), turned to 90 degrees
- moved D2 5.00 mm to (138.5, 74.7)
- moved D3 5.00 mm to (143.5, 74.7)
- moved R12 3.62 mm to (128.4, 106.6), turned to 90 degrees
- moved R13 1.60 mm to (157.1, 88.9)
Connections:
- D1 pad 1: GND1 -> GND
- D2 pad 1: GND1 -> GND
- D3 pad 1: GND1 -> GND
- D4 pad 1: GND1 -> GND
- J10 pad 1: GND1 -> GND
- J11 pad 1: GND1 -> GND
- J11 pad 5: /AI1 -> /AI1m
- J11 pad 6: /AI0 -> /AI0m
- R1 pad 2: Net-(D1-A) -> Net-(D4-A)
- R4 pad 2: Net-(D2-A) -> Net-(D3-A)
- R7 pad 2: Net-(D3-A) -> Net-(D2-A)
- R8 pad 2: Net-(D4-A) -> Net-(D1-A)
Routing:
- net GND1: track 146.9 -> 0.00 mm, vias 2 -> 0
- net GND: track 106.9 -> 191.4 mm
- net /AI0m: track 0.00 -> 68.1 mm, vias 0 -> 2
- net +5V: track 154.9 -> 87.7 mm, vias 2 -> 8
- net /AI0: track 75.1 -> 17.6 mm, vias 2 -> 0
- net /AI1m: track 0.00 -> 55.5 mm, vias 0 -> 2
- net /AI1: track 72.1 -> 17.3 mm, vias 2 -> 0
- net /DI1m: track 18.2 -> 27.2 mm
- net /DI2m: track 19.4 -> 26.1 mm
- net Net-(Q4-B): track 9.95 -> 4.62 mm
- net VDD: track 82.5 -> 77.7 mm
- net /DI0m: track 23.4 -> 26.8 mm
- net Net-(Q2-B): track 4.68 -> 5.58 mm
- net Net-(Q3-B): track 5.93 -> 5.09 mm
- net Net-(D5-A): track 5.29 -> 5.91 mm
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- added copper zone on B.Cu, net GND
- added copper zone on F.Cu, net GND
- removed copper zone on B.Cu, net (none)
Other:
- board text added: "+ - 24V"
- board text added: "+24V GND"
- board text added: "+5V GND"
- board text added: "+V5 GND VDD GND"
- board text added: "A1 A0"
- board text added: "A1 A0 D3 D2 D1 D0"
- board text added: "D0 D1 D2 D3 A0 A1"
- board text added: "DI3 DI2 DI1 DI0"
- board text added: "Designed by ODI"
- board text added: "GND VDD GND +5V"
