File: PPDuino_Nano_Electronic/V0.2/Entradas/PPDuino Nano Entradas.kicad_sch (KiCad schematic)
At the start: 26 parts, among them J10 PWR_OUT, J11 INPUTS, J2 DI, J3 AI, Q1 BC548, U1 4N35, U2 4N35, U3 4N35

Commit message: PCB V0.2
Parts:
- removed U1, U2, U3: 4N35, Package_DIP:DIP-6_W7.62mm_LongPads, symbol Isolator:4N35
- added D6, D7: Z5.1V, Diode_THT:D_DO-35_SOD27_P7.62mm_Horizontal, symbol Device:D_Zener
- added Q2, Q3, Q4: BC548, Package_TO_SOT_THT:TO-92L_Inline_Wide, symbol Transistor_BJT:BC548
- added R14, R15, R16, R17: 2.2k, Resistor_THT:R_Axial_DIN0207_L6.3mm_D2.5mm_P7.62mm_Horizontal, symbol Device:R
- renumbered D4 to D1, D3 to D2, D2 to D3, D1 to D4
Connections:
- net +5V: now also Q2.1 (C), Q3.1 (C), Q4.1 (C)
- net AI0: now also R15.1; no longer J11.6 (Pin_6)
- net AI1: now also R17.1; no longer J11.5 (Pin_5)
- net DI1m: now also Q2.3 (E)
- net DI2m: now also Q3.3 (E)
- net DI3m: now also Q4.3 (E)
- net GND: now also D6.2 (A), D7.2 (A), R14.2, R16.2
- net at R9.2: now also Q2.2 (B)
- net at R5.2: now also Q3.2 (B)
- net at R2.2: now also Q4.2 (B)
- new net AI0m: D6.1 (K), J11.6 (Pin_6), R14.1, R15.2
- new net AI1m: D7.1 (K), J11.5 (Pin_5), R16.1, R17.2
- no-connect marks 3 -> 0
Other:
- moved on the sheet: D1, D2, D3, D4, D5, Q1, R1, R10, R11, R12, R13, R2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
