File: PPDuino_Nano_Electronic/V0.2/Procesador/PPDuino_Nano_Procesador.kicad_pcb (KiCad board)
At the start: 2 copper layers, 39.7 x 71.8 mm, 10 parts, among them J1 PWR_IN, J11 INPUTS, J12 OUTPUTS, J2 Conn_01x12, U1 L7805, U6 +5V

Commit message: PCB V0.2
Parts:
- added G***: LOGO, Logo PPDuino Nano:Logo PPDuino Nano, F.Cu at (113.7, 64.1)
- added G***: LOGO, Logo Fab Lab PPD Electronica:Logo Fab Lab PPD Electronica, F.Cu at (100.5, 75.0)
- added G***: LOGO, Logo Fab Lab PPD Electronica:Logo Fab Lab PPD Electronica, B.Cu at (100.4, 84.0)
- added G***: LOGO, Logo PPDuino Nano:Logo PPDuino Nano, B.Cu at (100.5, 66.4)
Connections:
- A1 pad 25: /AI1 -> /AI1m
- A1 pad 26: /AI0 -> /AI0m
- C1 pad 2: GND1 -> GND
- J1 pad 1: GND1 -> GND
- J11 pad 1: GND1 -> GND
- J11 pad 10: /AI0 -> /DI0m
- J11 pad 5: /DI0m -> /AI1m
- J11 pad 6: /DI1m -> /AI0m
- J11 pad 7: /DI2m -> /DI3m
- J11 pad 8: /DI3m -> /DI2m
- J11 pad 9: /AI1 -> /DI1m
- J12 pad 1: GND1 -> GND
- J2 pad 1: GND1 -> GND
- J2 pad 3: +5V -> GND
- J2 pad 4: GND -> +5V
- U6 pad 2: GND1 -> GND
Routing:
- net GND: track 155.9 -> 269.7 mm, vias 6 -> 8
- net GND1: track 107.6 -> 0.00 mm
- net /AI1: track 47.4 -> 0.00 mm
- net /AI1m: track 0.00 -> 46.5 mm
- net /AI0: track 44.7 -> 0.00 mm
- net /AI0m: track 0.00 -> 42.8 mm
- net /DI0m: track 62.2 -> 76.9 mm, vias 0 -> 2
- net /DI1m: track 60.3 -> 70.4 mm, vias 0 -> 2
- net /DI2m: track 58.1 -> 64.8 mm, vias 0 -> 2
- net +5V: track 162.5 -> 157.9 mm, vias 6 -> 4
- net /DI3m: track 56.0 -> 59.5 mm, vias 0 -> 2
- net /SCK: track 35.2 -> 35.7 mm
- added copper zone on B.Cu, net GND
- added copper zone on F.Cu, net GND
- removed copper zone on B.Cu, net (none)
Other:
- board text added: "+ 24V -"
- board text added: "+5V GND VDD GND"
- board text added: "- 24V +"
- board text added: "A1 A0 D3 D2 D1 D0"
- board text added: "D0 D1 D2 D3 A0 A1"
- board text added: "D0 D1 D2 D3 R0 R1"
- board text added: "Designed by ODI"
- board text added: "GND VDD GND +5V"
- board text added: "MOSI MISO SCK"
- board text added: "R1 R0 D3 D2 D1 D0"
- board text added: "RX TX SS"
- board text added: "SCK MISO MOSI"
- board text added: "SCL SDA"
- board text added: "SDA SCL"
- board text added: "SS TX RX"
