File: PPDuino_Nano_Electronic/V0.2/Procesador/PPDuino_Nano_Procesador.kicad_sch (KiCad schematic)
At the start: 9 parts, among them J1 PWR_IN, J11 INPUTS, J12 OUTPUTS, J2 Conn_01x12, U1 L7805, U6 +5V

Commit message: PCB V0.2
Connections:
- net GND1 is gone; now on net GND: C1.2, J1.1 (Pin_1), J11.1 (Pin_1), J12.1 (Pin_1), J2.1 (Pin_1), U6.2 (-IN)
- net +5V: now also J2.4 (Pin_4); no longer J2.3 (Pin_3)
- net DI0m: now also J11.10 (Pin_10); no longer J11.5 (Pin_5)
- net DI1m: now also J11.9 (Pin_9); no longer J11.6 (Pin_6)
- net DI2m: now also J11.8 (Pin_8); no longer J11.7 (Pin_7)
- net DI3m: now also J11.7 (Pin_7); no longer J11.8 (Pin_8)
- net GND: now also J2.3 (Pin_3); no longer J2.4 (Pin_4)
- net AI0 renamed AI0m
- net AI0m: now also J11.6 (Pin_6); no longer J11.10 (Pin_10)
- net AI1 renamed AI1m
- net AI1m: now also J11.5 (Pin_5); no longer J11.9 (Pin_9)
