File: PPDuino_Nano_Electronic/V0.2/Salidas/PPDuino Nano Salidas.kicad_pcb (KiCad board)
At the start: 2 copper layers, 51.6 x 92.8 mm, 29 parts, among them J12 OUTPUTS, J13 SEL1, J14 RLY0, J6 SEL0, J7 RLY1, J8 PWM, J9 PWR_OUT, Q1 BC548, Q2 BC548, U5 L293D

Commit message: PCB V0.2
Parts:
- added G***: LOGO, Logo Fab Lab PPD Electronica:Logo Fab Lab PPD Electronica, F.Cu at (159.9, 58.0)
- added G***: LOGO, Logo PPDuino Nano:Logo PPDuino Nano, F.Cu at (125.6, 94.4)
- added G***: LOGO, Logo Fab Lab PPD Electronica:Logo Fab Lab PPD Electronica, B.Cu at (159.9, 58.0)
- added G***: LOGO, Logo PPDuino Nano:Logo PPDuino Nano, B.Cu at (125.6, 94.4)
- D6, D8: value 1N4148 -> 4148
Routing:
- added copper zone on B.Cu, net GND
- added copper zone on F.Cu, net GND
- removed copper zone on B.Cu, net (none)
Other:
- board text added: "+5V GND VDD GND"
- board text added: "D0 D1 D2 D3 R0 R1"
- board text added: "DO0 DO1 DO2 DO3"
- board text added: "DO3 DO2 DO1 DO0"
- board text added: "Designed by ODI"
- board text added: "GND VDD"
- board text added: "GND VDD GND +5V"
- board text added: "R0 R0 R1 R1"
- board text added: "R1 R0 D3 D2 D1 D0"
- board text added: "R1 R1 R0 R0"
- board text added: "VDD GND"
